Commit message: add rrt navigation

File: xacro/F11Robo.xacro (robot description, xacro)
@@ -1,132 +1,134 @@
 <?xml version="1.0"?>
 <robot name="F11Robot" xmlns:xacro="http://ros.org/wiki/xacro">
-  <material name="gray">
-    <color rgba="0.5 0.5 0.5 2.5"/>
-  </material>
-  <material name="red">
-    <color rgba="1.0 0.0 0.0 2.5"/>
-  </material>
-  <xacro:macro name="wheel_macro" params="parent prefix xyz deg　*joint_axis">
-    <joint name="${prefix}_joint" type="continuous">
-      <origin xyz="${xyz}" rpy="0 0 ${radians(deg)}"/>
-      <parent link="${parent}"/>
-      <child  link="${prefix}_link"/>
-      <insert_block name="joint_axis"/>
-    </joint>
-    <transmission name="${prefix}_trans">
-      <type>transmission_interface/SimpleTransmission</type>
-      <joint name="${prefix}_joint">
-          <hardwareInterface>hardware_interface/VelocityJointInterface</hardwareInterface>
-      </joint>
-      <actuator name="${prefix}_motor">
-        <hardwareInterface>hardware_interface/VelocityJointInterface</hardwareInterface>
-        <mechanismReduction>1</mechanismReduction>
-      </actuator>
-    </transmission>
-    <link name="${prefix}_link">
-      <inertial>
-        <origin xyz="0 0 0" rpy="0 0 0"/>
-        <mass value="0.1"/>
-        <inertia ixx="0.0001" ixy="0.0" ixz="0.0" iyy="0.0001" iyz="0.0" izz="0.0001"/>
-      </inertial>
-      <visual>
-        <geometry>
-          <mesh filename="package://F11Robo/stl/Robo_wheel.stl"/>
-        </geometry>
-        <material name="red"/>
-      </visual>
-      <collision>
-        <geometry>
-          <cylinder radius="0.03336" length="0.02" />
-        </geometry>
-      </collision>
-    </link>
-    <gazebo reference="${prefix}_link">
-      <material>Gazebo/Red</material>
-      <mu1 value="2.5" />
-      <mu2 value="2.5" />
-      <kp value="50000" />
-      <kd value="10" />
-    </gazebo>
-  </xacro:macro>
-  <xacro:macro name="ball_macro" params="prefix xyz">
-    <joint name="${prefix}_joint" type="fixed">
-      <origin xyz="${xyz}" rpy="0 0 0"/>
-      <parent link="base_link"/>
-      <child  link="${prefix}_link"/>
-      <axis xyz="0 0 1" />
-    </joint>
-    <link name="${prefix}_link">
-      <origin xyz="0 0 0" rpy="0 0 0" />
-      <visual>
-        <geometry>
-          <sphere radius="0.005" />
-        </geometry>
-        <material name="red"/>
-      </visual>
-      <collision>
-        <geometry>
-          <sphere radius="0.005" />
-        </geometry>
-        <material name="red" />
-      </collision>
-    </link>
-    <gazebo reference="${prefix}_link">
-      <material>Gazebo/Red</material>
-      <mu1 value="0.1" />
-      <mu2 value="0.1" />
-    </gazebo>
-  </xacro:macro>
-  <link name="base_link"/>
-  <joint name="body_joint" type="fixed">
-    <parent link="base_link"/>
-    <child  link="body_link"/>
-    <origin xyz="0 0 0.0033" rpy="0 0 0"/>
-  </joint>
-  <link name="body_link">
-    <inertial>
-      <origin xyz="0 0 0" rpy="0 0 0"/>
-      <mass value="1.0"/>
-      <inertia ixx="0.001" ixy="0.0" ixz="0.0" iyy="0.001" iyz="0.0" izz="0.001"/>
-    </inertial>
-    <visual>
-      <origin xyz="0 0 0" rpy="0 0 0" />
-      <geometry>
-        <mesh filename="package://F11Robo/stl/Robo_body.stl"/>
-      </geometry>
-      <material name="gray" />
-    </visual>
-    <collision>
-      <origin xyz="0 0 0" rpy="0 0 0" />
-      <geometry>
-        <box size="0.24 0.23 0.0032" />
-      </geometry>
-    </collision>
-  </link>
-  <gazebo reference="body_link">
-    <material>Gazebo/Gray</material>
-  </gazebo>
-  <xacro:wheel_macro prefix="left_wheel"  parent="base_link" xyz="0 0.1 0.03335" deg="180">
-    <axis xyz="0 -1 0"/>
-  </xacro:wheel_macro>
-  <xacro:wheel_macro prefix="right_wheel" parent="base_link" xyz="0 -0.1 0.03335" deg="0">
-    <axis xyz="0 1 0"/>
-  </xacro:wheel_macro>
-  <xacro:ball_macro prefix="left_ball" xyz="-0.155 0.0755 0.005"/>
-  <xacro:ball_macro prefix="right_ball" xyz="-0.155 -0.0755 0.005"/>
-  <gazebo>
-    <plugin name="gazebo_ros_control" filename="libgazebo_ros_control.so">
-      <robotNamespace>/F11Robo</robotNamespace>
-      <robotSimType>gazebo_ros_control/DefaultRobotHWSim</robotSimType>
-      <legacyModeNS>true</legacyModeNS>
-    </plugin>
-  </gazebo>
-  <gazebo>
-    <plugin name="ground_truth" filename="libgazebo_ros_p3d.so">
-      <frameName>world</frameName>
-      <bodyName>base_link</bodyName>
-      <topicName>/tracker</topicName>
-      <updateRate>10.0</updateRate>
-    </plugin>
-  </gazebo>
+	<material name="gray">
+		<color rgba="0.7 0.7 0.7 2.5"/>
+	</material>
+	<material name="red">
+		<color rgba="1.0 0.0 0.0 2.5"/>
+	</material>
+	<xacro:macro name="wheel_macro" params="parent prefix xyz deg　*joint_axis">
+		<joint name="${prefix}_joint" type="continuous">
+		<origin xyz="${xyz}" rpy="0 0 ${radians(deg)}"/>
+		<parent link="${parent}"/>
+		<child  link="${prefix}_link"/>
+		<insert_block name="joint_axis"/>
+		</joint>
+		<transmission name="${prefix}_trans">
+		<type>transmission_interface/SimpleTransmission</type>
+		<joint name="${prefix}_joint">
+			<hardwareInterface>hardware_interface/VelocityJointInterface</hardwareInterface>
+		</joint>
+		<actuator name="${prefix}_motor">
+			<hardwareInterface>hardware_interface/VelocityJointInterface</hardwareInterface>
+			<mechanismReduction>1</mechanismReduction>
+		</actuator>
+		</transmission>
+		<link name="${prefix}_link">
+		<inertial>
+			<origin xyz="0 0 0" rpy="0 0 0"/>
+			<mass value="0.1"/>
+			<inertia ixx="0.0001" ixy="0.0" ixz="0.0" iyy="0.0001" iyz="0.0" izz="0.0001"/>
+		</inertial>
+		<visual>
+			<geometry>
+			<mesh filename="package://F11Robo/stl/Robo_wheel.stl"/>
+			</geometry>
+			<material name="red"/>
+		</visual>
+		<collision>
+			<geometry>
+			<cylinder radius="0.03336" length="0.011" />
+			</geometry>
+		</collision>
+		</link>
+		<gazebo reference="${prefix}_link">
+		<material>Gazebo/Red</material>
+		<mu1 value="3.0" />
+		<mu2 value="3.0" />
+		<kp value="50000" />
+		<kd value="10" />
+		</gazebo>
+	</xacro:macro>
+	<xacro:macro name="ball_macro" params="prefix xyz">
+		<joint name="${prefix}_joint" type="fixed">
+		<origin xyz="${xyz}" rpy="0 0 0"/>
+		<parent link="base_link"/>
+		<child  link="${prefix}_link"/>
+		<axis xyz="0 0 1" />
+		</joint>
+		<link name="${prefix}_link">
+		<origin xyz="0 0 0" rpy="0 0 0" />
+		<visual>
+			<geometry>
+			<sphere radius="0.005" />
+			</geometry>
+			<material name="red"/>
+		</visual>
+		<collision>
+			<geometry>
+			<sphere radius="0.005" />
+			</geometry>
+			<material name="red" />
+		</collision>
+		</link>
+		<gazebo reference="${prefix}_link">
+		<material>Gazebo/Red</material>
+		<mu1 value="0.2" />
+		<mu2 value="0.2" />
+		</gazebo>
+	</xacro:macro>
+	<link name="base_link"/>
+	<joint name="body_joint" type="fixed">
+		<parent link="base_link"/>
+		<child  link="body_link"/>
+		<origin xyz="0 0 0.0033" rpy="0 0 0"/>
+	</joint>
+	<link name="body_link">
+		<inertial>
+		<origin xyz="0 0 0" rpy="0 0 0"/>
+		<mass value="1.0"/>
+		<inertia ixx="0.001" ixy="0.0" ixz="0.0" iyy="0.001" iyz="0.0" izz="0.001"/>
+		</inertial>
+		<visual>
+		<origin xyz="0 0 0" rpy="0 0 0" />
+		<geometry>
+			<mesh filename="package://F11Robo/stl/Robo_body.stl"/>
+		</geometry>
+		<material name="gray" />
+		</visual>
+		<collision>
+		<origin xyz="0 0 0" rpy="0 0 0" />
+		<geometry>
+			<box size="0.24 0.23 0.005" />
+		</geometry>
+		</collision>
+	</link>
+	<gazebo reference="body_link">
+		<material>Gazebo/Gray</material>
+		<mu1 value="0.3" />
+		<mu2 value="0.3" />
+	</gazebo>
+	<xacro:wheel_macro prefix="left_wheel"  parent="base_link" xyz="0 0.1 0.03335" deg="180">
+		<axis xyz="0 -1 0"/>
+	</xacro:wheel_macro>
+	<xacro:wheel_macro prefix="right_wheel" parent="base_link" xyz="0 -0.1 0.03335" deg="0">
+		<axis xyz="0 1 0"/>
+	</xacro:wheel_macro>
+	<xacro:ball_macro prefix="left_ball" xyz="-0.155 0.0755 0.005"/>
+	<xacro:ball_macro prefix="right_ball" xyz="-0.155 -0.0755 0.005"/>
+	<gazebo>
+		<plugin name="gazebo_ros_control" filename="libgazebo_ros_control.so">
+		<robotNamespace>/F11Robo</robotNamespace>
+		<robotSimType>gazebo_ros_control/DefaultRobotHWSim</robotSimType>
+		<legacyModeNS>true</legacyModeNS>
+		</plugin>
+	</gazebo>
+	<gazebo>
+		<plugin name="ground_truth" filename="libgazebo_ros_p3d.so">
+		<frameName>world</frameName>
+		<bodyName>base_link</bodyName>
+		<topicName>/tracker</topicName>
+		<updateRate>10.0</updateRate>
+		</plugin>
+	</gazebo>
 </robot>

Commit message: update Robo model

File: xacro/F11Robo.xacro (robot description, xacro)
@@ -8,73 +8,80 @@
 		<color rgba="1.0 0.0 0.0 2.5"/>
 	</material>
+	<material name="blue">
+		<color rgba="0.0 0.0 1.0 2.5"/>
+	</material>
 	<xacro:macro name="wheel_macro" params="parent prefix xyz deg　*joint_axis">
 		<joint name="${prefix}_joint" type="continuous">
-		<origin xyz="${xyz}" rpy="0 0 ${radians(deg)}"/>
-		<parent link="${parent}"/>
-		<child  link="${prefix}_link"/>
-		<insert_block name="joint_axis"/>
+			<origin xyz="${xyz}" rpy="0 0 ${radians(deg)}"/>
+			<parent link="${parent}"/>
+			<child  link="${prefix}_link"/>
+			<insert_block name="joint_axis"/>
 		</joint>
 		<transmission name="${prefix}_trans">
-		<type>transmission_interface/SimpleTransmission</type>
-		<joint name="${prefix}_joint">
-			<hardwareInterface>hardware_interface/VelocityJointInterface</hardwareInterface>
-		</joint>
-		<actuator name="${prefix}_motor">
-			<hardwareInterface>hardware_interface/VelocityJointInterface</hardwareInterface>
-			<mechanismReduction>1</mechanismReduction>
-		</actuator>
+			<type>transmission_interface/SimpleTransmission</type>
+			<joint name="${prefix}_joint">
+				<hardwareInterface>hardware_interface/VelocityJointInterface</hardwareInterface>
+			</joint>
+			<actuator name="${prefix}_motor">
+				<hardwareInterface>hardware_interface/VelocityJointInterface</hardwareInterface>
+				<mechanismReduction>1</mechanismReduction>
+			</actuator>
 		</transmission>
 		<link name="${prefix}_link">
-		<inertial>
-			<origin xyz="0 0 0" rpy="0 0 0"/>
-			<mass value="0.1"/>
-			<inertia ixx="0.0001" ixy="0.0" ixz="0.0" iyy="0.0001" iyz="0.0" izz="0.0001"/>
-		</inertial>
-		<visual>
-			<geometry>
-			<mesh filename="package://F11Robo/stl/Robo_wheel.stl"/>
-			</geometry>
-			<material name="red"/>
-		</visual>
-		<collision>
-			<geometry>
-			<cylinder radius="0.03336" length="0.011" />
-			</geometry>
-		</collision>
+			<inertial>
+				<origin xyz="0 0 0" rpy="0 0 0"/>
+				<mass value="0.2"/>
+				<inertia ixx="0.0001" ixy="0.0" ixz="0.0" iyy="0.0001" iyz="0.0" izz="0.0001"/>
+			</inertial>
+			<visual>
+				<origin xyz="0 0 0" rpy="0 0 0"/>
+				<geometry>
+					<mesh filename="package://F11Robo/stl/Robo_wheel.stl"/>
+				</geometry>
+				<material name="red"/>
+			</visual>
+			<collision>
+				<origin xyz="0 0 0" rpy="${radians(90)} 0 0"/>
+				<geometry>
+					<cylinder radius="0.03336" length="0.011" />
+				</geometry>
+			</collision>
 		</link>
 		<gazebo reference="${prefix}_link">
-		<material>Gazebo/Red</material>
-		<mu1 value="3.0" />
-		<mu2 value="3.0" />
-		<kp value="50000" />
-		<kd value="10" />
+			<material>Gazebo/Red</material>
+			<mu1 value="3.0" />
+			<mu2 value="3.0" />
+			<kp value="50000" />
+			<kd value="10" />
 		</gazebo>
 	</xacro:macro>
 	<xacro:macro name="ball_macro" params="prefix xyz">
 		<joint name="${prefix}_joint" type="fixed">
-		<origin xyz="${xyz}" rpy="0 0 0"/>
-		<parent link="base_link"/>
-		<child  link="${prefix}_link"/>
-		<axis xyz="0 0 1" />
+			<origin xyz="${xyz}" rpy="0 0 0"/>
+			<parent link="base_link"/>
+			<child  link="${prefix}_link"/>
 		</joint>
 		<link name="${prefix}_link">
-		<origin xyz="0 0 0" rpy="0 0 0" />
-		<visual>
-			<geometry>
-			<sphere radius="0.005" />
-			</geometry>
-			<material name="red"/>
-		</visual>
-		<collision>
-			<geometry>
-			<sphere radius="0.005" />
-			</geometry>
-			<material name="red" />
-		</collision>
+			<visual>
+				<origin xyz="0 0 0" rpy="0 0 0" />
+				<geometry>
+					<sphere radius="0.005" />
+				</geometry>
+				<material name="red"/>
+			</visual>
+			<collision>
+				<origin xyz="0 0 0" rpy="0 0 0" />
+				<geometry>
+					<sphere radius="0.005" />
+				</geometry>
+				<material name="red" />
+			</collision>
 		</link>
 		<gazebo reference="${prefix}_link">
-		<material>Gazebo/Red</material>
-		<mu1 value="0.2" />
-		<mu2 value="0.2" />
+			<material>Gazebo/Red</material>
+			<mu1 value="0.0" />
+			<mu2 value="0.0" />
+			<mass value="0.1" />
+			<inertia ixx="0.0001" ixy="0.0" ixz="0.0" iyy="0.0001" iyz="0.0" izz="0.0001"/>
 		</gazebo>
 	</xacro:macro>
@@ -87,26 +94,26 @@
 	<link name="body_link">
 		<inertial>
-		<origin xyz="0 0 0" rpy="0 0 0"/>
-		<mass value="1.0"/>
-		<inertia ixx="0.001" ixy="0.0" ixz="0.0" iyy="0.001" iyz="0.0" izz="0.001"/>
+			<origin xyz="-0.05 0 0.03" rpy="0 0 0" />
+			<mass value="1.0"/>
+			<inertia ixx="0.001" ixy="0.0" ixz="0.0" iyy="0.001" iyz="0.0" izz="0.001"/>
 		</inertial>
 		<visual>
-		<origin xyz="0 0 0" rpy="0 0 0" />
-		<geometry>
-			<mesh filename="package://F11Robo/stl/Robo_body.stl"/>
-		</geometry>
-		<material name="gray" />
+			<origin xyz="0 0 0" rpy="0 0 0" />
+			<geometry>
+				<mesh filename="package://F11Robo/stl/Robo_body.stl"/>
+			</geometry>
+			<material name="gray" />
 		</visual>
 		<collision>
-		<origin xyz="0 0 0" rpy="0 0 0" />
-		<geometry>
-			<box size="0.24 0.23 0.005" />
-		</geometry>
+			<origin xyz="-0.05 0 0.03" rpy="0 0 0" />
+			<geometry>
+				<box size="0.24 0.23 0.05" />
+			</geometry>
 		</collision>
 	</link>
 	<gazebo reference="body_link">
 		<material>Gazebo/Gray</material>
-		<mu1 value="0.3" />
-		<mu2 value="0.3" />
+		<mu1>0.05</mu1>
+		<mu2>0.05</mu2>
 	</gazebo>
 	<xacro:wheel_macro prefix="left_wheel"  parent="base_link" xyz="0 0.1 0.03335" deg="180">
@@ -118,5 +125,5 @@
 	<xacro:ball_macro prefix="left_ball" xyz="-0.155 0.0755 0.005"/>
 	<xacro:ball_macro prefix="right_ball" xyz="-0.155 -0.0755 0.005"/>
-	<xacro:laser_macro prefix="front_laser" parent="base_link" xyz="0.05 0 0.078"/>
+	<xacro:laser_macro prefix="laser" parent="base_link" xyz="0.05 0 0.078"/>
 	<gazebo>
 		<plugin name="gazebo_ros_control" filename="libgazebo_ros_control.so">

File: xacro/lidar.xacro (robot description, xacro)
@@ -12,15 +12,15 @@
 			<cylinder radius="0.0329" length="0.04" />
 			</geometry>
-			<material name="red" />
+			<material name="blue" />
 		</visual>
 		<collision>
 			<origin xyz="0 0 0" rpy="0 0 0"/>
 			<geometry>
-			<cylinder radius="0.02" length="0.06" />
+			<cylinder radius="0.0329" length="0.04" />
 			</geometry>
 		</collision>
 		</link>
 		<gazebo reference="${prefix}_link">
-		<material>Gazebo/Red</material>
+		<material>Gazebo/Blue</material>
 		<sensor type="ray" name="${prefix}">
 			<pose>0 0 0 0 0 0</pose>
